File: src/Telerob_hardware/Motor_driver/Motor_Driver.kicad_sch (KiCad schematic)
At the start: 22 parts

Commit message: Circ 2
Parts:
- JCAN1: footprint (none) -> Connector_PinHeader_2.54mm:PinHeader_1x07_P2.54mm_Vertical
Changed lines of the file:
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@@
 			)
 		)
-		(property "Footprint" ""
+		(property "Footprint" "Connector_PinHeader_2.54mm:PinHeader_1x07_P2.54mm_Vertical"
 			(at 189.23 61.595 0)
 			(effects

Commit message: PCB_act
Connections:
- net GP16 is gone; now on net SO: Pi1.20 (GP16)
- net GP17 is gone; now on net CS: Pi1.21 (GP17)
- net GP18 is gone; now on net SCK: Pi1.23 (GP18)
- net GP19 is gone; now on net SI: Pi1.24 (GP19)
- net GP20 is gone; now on net INT: Pi1.25 (GP20)
- net GP26 is gone; now on net VML: Pi1.30 (GP26)
Other:
- moved on the sheet: Pi1

Commit message: Codes
Parts:
- added Pins1: ~, Connector_PinHeader_2.54mm:PinHeader_1x04_P2.54mm_Vertical, symbol Connector_Generic:Conn_01x04
Connections:
- net GP7 is gone; now on net A_1: Pi1.9 (GP7)
- net GP8 is gone; now on net B_1: Pi1.10 (GP8)
- net 3V3_O: now also JM1.4 (Pin_4), JM2.4 (Pin_4); no longer JM1.2 (Pin_2), JM2.2 (Pin_2)
- net A_2: now also Pi1.3 (GP2)
- net B_2: now also Pi1.4 (GP3)
- net GP10: now also Pins1.1 (Pin_1)
- net GP11: now also Pins1.2 (Pin_2)
- net GP12: now also Pins1.3 (Pin_3)
- net GP13: now also Pins1.4 (Pin_4)
- net GP21: now also JS1.1 (Pin_1)
- net GP22: now also JM1.2 (Pin_2)
- net GP4: now also JM2.2 (Pin_2); no longer JM1.1 (Pin_1)
- net GP5: now also JM2.1 (Pin_1); no longer JM1.4 (Pin_4), JS1.1 (Pin_1)
- net GP9: now also JM1.1 (Pin_1)
- removed net GP2: JM2.1 (Pin_1), Pi1.3 (GP2)
- removed net GP3: JM2.4 (Pin_4), Pi1.4 (GP3)
Changed lines of the file:
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@@
 	(wire
 		(pts
+			(xy 181.61 74.295) (xy 184.15 74.295)
+		)
+		(stroke
+			(width 0)
+			(type default)
+		)
+	)
+	(wire
+		(pts
 			(xy 76.2 43.815) (xy 73.66 43.815)
 		)
@@
 	(wire
 		(pts
+			(xy 181.61 81.915) (xy 184.15 81.915)
+		)
+		(stroke
+			(width 0)
+			(type default)
+		)
+	)
+	(wire
+		(pts
 			(xy 78.74 90.17) (xy 76.835 90.17)
 		)
@@
 	(wire
 		(pts
+			(xy 181.61 79.375) (xy 184.15 79.375)
+		)
+		(stroke
+			(width 0)
+			(type default)
+		)
+	)
+	(wire
+		(pts
 			(xy 109.22 98.425) (xy 111.76 98.425)
 		)
@@
 	(wire
 		(pts
+			(xy 181.61 76.835) (xy 184.15 76.835)
+		)
+		(stroke
+			(width 0)
+			(type default)
+		)
+	)
+	(wire
+		(pts
 			(xy 149.86 60.96) (xy 152.4 60.96)
 		)
@@
 		)
 	)
+	(hierarchical_label "GP12"
+		(shape input)
+		(at 181.61 79.375 180)
+		(effects
+			(font
+				(size 1.27 1.27)
+			)
+			(justify right)
+		)
+	)
 	(hierarchical_label "GP22"
 		(shape input)
@@
 		)
 	)
-	(hierarchical_label "GP3"
+	(hierarchical_label "B_2"
 		(shape input)
 		(at 76.2 59.055 0)
@@
 		)
 	)
-	(hierarchical_label "GP4"
+	(hierarchical_label "GP9"
 		(shape input)
 		(at 147.955 38.735 180)
@@
 		)
 	)
-	(hierarchical_label "GP3"
-		(shape input)
-		(at 165.735 25.4 0)
-		(effects
-			(font
-				(size 1.27 1.27)
-			)
-			(justify left)
-		)
-	)
 	(hierarchical_label "GND"
 		(shape input)
@@
 		)
 	)
+	(hierarchical_label "GP10"
+		(shape input)
+		(at 181.61 74.295 180)
+		(effects
+			(font
+				(size 1.27 1.27)
+			)
+			(justify right)
+		)
+	)
 	(hierarchical_label "GND"
 		(shape input)
@@
 		)
 	)
-	(hierarchical_label "GP5"
+	(hierarchical_label "GP21"
 		(shape input)
 		(at 109.22 88.265 180)
@@
 		)
 	)
-	(hierarchical_label "GP8"
+	(hierarchical_label "B_1"
 		(shape input)
 		(at 76.2 43.815 0)
@@
 		)
 	)
-	(hierarchical_label "GP2"
+	(hierarchical_label "GP11"
+		(shape input)
+		(at 181.61 76.835 180)
+		(effects
+			(font
+				(size 1.27 1.27)
+			)
+			(justify right)
+		)
+	)
+	(hierarchical_label "GP5"
 		(shape input)
 		(at 147.955 25.4 180)
@@
 		)
 	)
+	(hierarchical_label "GP13"
+		(shape input)
+		(at 181.61 81.915 180)
+		(effects
+			(font
+				(size 1.27 1.27)
+			)
+			(justify right)
+		)
+	)
 	(hierarchical_label "GND"
 		(shape input)
@@
 		)
 	)
-	(hierarchical_label "GP5"
+	(hierarchical_label "3V3_O"
 		(shape input)
 		(at 165.735 38.735 0)
@@
 		)
 	)
-	(hierarchical_label "3V3_O"
+	(hierarchical_label "GP4"
 		(shape input)
 		(at 147.955 27.94 180)
@@
 		)
 	)
-	(hierarchical_label "3V3_O"
+	(hierarchical_label "GP22"
 		(shape input)
 		(at 147.955 41.275 180)
@@
 		)
 	)
-	(hierarchical_label "GP2"
+	(hierarchical_label "A_2"
 		(shape input)
 		(at 76.2 61.595 0)
@@
 		)
 	)
+	(hierarchical_label "3V3_O"
+		(shape input)
+		(at 165.735 25.4 0)
+		(effects
+			(font
+				(size 1.27 1.27)
+			)
+			(justify left)
+		)
+	)
 	(hierarchical_label "GP28"
 		(shape input)
@@
 		)
 	)
-	(hierarchical_label "GP7"
+	(hierarchical_label "A_1"
 		(shape input)
 		(at 76.2 46.355 0)
@@
 					(unit 1)
 				)
+			)
+		)
+	)
+	(symbol
+		(lib_id "Connector_Generic:Conn_01x04")
+		(at 189.23 76.835 0)
+		(unit 1)
+		(exclude_from_sim no)
+		(in_bom yes)
+		(on_board yes)
+		(dnp no)
+		(fields_autoplaced yes)
+		(property "Reference" "Pins1"
+			(at 191.77 77.4699 0)
+			(effects
+				(font
+					(size 1.27 1.27)
+				)
+				(justify left)
+			)
+		)
+		(property "Value" "~"
+			(at 191.77 79.375 0)
+			(effects
+				(font
+					(size 1.27 1.27)
+				)
+				(justify left)
+			)
+		)
+		(property "Footprint" "Connector_PinHeader_2.54mm:PinHeader_1x04_P2.54mm_Vertical"
+			(at 189.23 76.835 0)
+			(effects
+				(font
+					(size 1.27 1.27)
+				)
+				(hide yes)
+			)
+		)
+		(property "Datasheet" "~"
+			(at 189.23 76.835 0)
+			(effects
+				(font
+					(size 1.27 1.27)
+				)
+				(hide yes)
+			)
+		)
+		(property "Description" "Generic connector, single row, 01x04, script generated (kicad-library-utils/schlib/autogen/connector/)"
+			(at 189.23 76.835 0)
+			(effects
+				(font
+					(size 1.27 1.27)
+				)
+				(hide yes)
+			)
+		)
+		(pin "2"
+		)
+		(pin "4"
+		)
+		(pin "1"
+		)
+		(pin "3"
+		)
+		(instances
+			(project "Motor_Driver"
+				(path "/22c889e8-9f1f-4928-aa68-6394d147a31f"
+					(reference "Pins1")
+					(unit 1)
+				)
